File: board/DMX512_LED_6Ch.kicad_sch (KiCad schematic)
At the start: 36 parts, among them J3 Conn_01x02, J6 Conn_ARM_JTAG_SWD_10, J7 Conn_01x04, SW1 SW_DIP_x10, SW2 SW_Push, U1 ATSAMD21G18A-A, Y1 32.768kHz

Commit message: doing some cost reduction
Parts:
- removed C2: 1uF, Capacitor_SMD:C_0402_1005Metric, symbol Device:C
- removed C6, C7: 22pF, Capacitor_SMD:C_0402_1005Metric, symbol Device:C
- removed J6: Conn_ARM_JTAG_SWD_10, Connector_PinHeader_1.27mm:PinHeader_2x05_P1.27mm_Vertical_SMD, symbol Connector:Conn_ARM_JTAG_SWD_10
- removed U1: ATSAMD21G18A-A, Package_QFP:TQFP-48_7x7mm_P0.5mm, symbol MCU_Microchip_SAMD:ATSAMD21G18A-A
- removed Y1: 32.768kHz, Crystal:Crystal_SMD_EuroQuartz_EQ161-2Pin_3.2x1.5mm, symbol Device:Crystal
- added J6: AVR-ISP-6, Connector:Tag-Connect_TC2030-IDC-NL_2x03_P1.27mm_Vertical, symbol Connector:AVR-ISP-6
- added J8: Conn_01x06, symbol Connector_Generic:Conn_01x06
- added U1: ATmega8A-A, Package_QFP:TQFP-32_7x7mm_P0.8mm, symbol MCU_Microchip_ATmega:ATmega8A-A
- added Y1: 16MHz, Crystal:Resonator_SMD_Murata_CSTxExxV-3Pin_3.0x1.1mm, symbol Device:Resonator
Connections:
- net +3V3: no longer C3.1, C4.1, C5.1, C8.1, R6.1, R7.1
- net CH1_BLU_EN: now also U1.10 (PD6)
- net CH1_GRN_EN: now also U1.9 (PD5)
- net CH1_RED_EN: now also U1.1 (PD3)
- net DMX_DIR: now also U1.32 (PD2)
- net DMX_IN: now also U1.30 (PD0)
- net DMX_OUT: now also U1.31 (PD1)
- net GND: now also J6.6 (GND), U1.21 (AGND), U1.3 (GND), U1.5 (GND), Y1.2
- net I2C_SCL: now also U1.28 (PC5)
- net I2C_SDA: now also U1.27 (PC4)
- net TMP_MON: now also U1.19 (ADC6)
- net VCC_MON: now also U1.22 (ADC7)
- net ~{RESET}: now also J6.5 (~{RST}), U1.29 (PC6/~{RESET})
- net LED2: now reaches R9.1
- net LED3: now reaches R10.1
- net LED1: now reaches R8.1
- new net: U1.7 (PB6/XTAL1), Y1.1
- new net: U1.8 (PB7/XTAL2), Y1.3
- new net +5V: C3.1, C4.1, C5.1, C8.1, J6.2 (VCC), R6.1, R7.1, U1.18 (AVCC), U1.4 (VCC), U1.6 (VCC)
- new net MISO: J6.1 (MISO), U1.16 (PB4)
- new net MOSI: J6.4 (MOSI), U1.15 (PB3)
- new net SCK: J6.3 (SCK), U1.17 (PB5)
- no-connect marks 2 -> 0
Other:
- sheet COMS ports: added none; removed USB_D_N, USB_D_P
- moved on the sheet: C10, C3, C4, C5, C8, C9, D2, D3, D4, D5, D6, H4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
